File: PCB/LED driver/LED driver.kicad_pcb (KiCad board)
At the start: 2 copper layers, 91.4 x 53.8 mm, 69 parts, among them J1 Conn_01x04, J10 Conn_01x04, J11 Conn_01x04, J12 Conn_01x04, J13 Conn_01x04, J14 Conn_01x04, J2 Conn_01x02, J3 Conn_01x04, J4 Conn_01x04, J5 Conn_01x04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

Commit message: 20230317-1646-laptop
Parts:
- moved R7 60.4 mm to (162.8, 102.4)
- moved R5 53.5 mm to (162.8, 106.4)
- moved R8 50.2 mm to (162.8, 100.3)
- moved R6 47.3 mm to (162.8, 104.4)
- moved R9 38.7 mm to (162.8, 98.3)
- moved J1 26.1 mm to (175.9, 81.8), turned to 90 degrees
- moved R4 25.5 mm to (162.8, 108.5)
Routing:
- net +5VD: track 0.00 -> 113.6 mm, vias 0 -> 1
- net SDA: track 0.00 -> 91.9 mm
- net SCL: track 0.00 -> 88.6 mm
- net B1: track 0.00 -> 39.5 mm, vias 0 -> 4
- net G1: track 0.00 -> 35.3 mm, vias 0 -> 4
- net +5V: track 113.6 -> 146.1 mm
- net R1: track 0.00 -> 31.1 mm, vias 0 -> 4
- net GND: track 223.2 -> 252.8 mm
- net Net-(J4-Pad2): track 0.00 -> 25.4 mm
- net Net-(J4-Pad3): track 0.00 -> 23.9 mm
- net Net-(J4-Pad4): track 0.00 -> 22.4 mm
- net Net-(J3-Pad2): track 0.00 -> 16.5 mm
- net Net-(J3-Pad3): track 0.00 -> 15.0 mm
- net Net-(J3-Pad4): track 0.00 -> 13.1 mm
- net Net-(J5-Pad4): track 0.00 -> 5.35 mm
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Other:
- board size 91.4 x 53.8 mm -> 98.6 x 53.8 mm
- board text added: "5V(Arduino)"
- board text added: "LED power"
- board text added: "SCL"
- board text added: "SDA"
